File: Hardware/SparkFun_Serial_MP3_Player_Shield_MY1690X.kicad_pcb (KiCad board)
At the start: 2 copper layers, 53.3 x 59.7 mm, 77 parts, among them J1 3.5mm TRRS, J3 Conn_01x03, J4 USB_C_Receptacle, J6 microSD, Q1 BSS138, SW1 SMD_5.2x5.2mm_h2.5mm, U2 MY1690X

Commit message: Add Busy LED, inline caps to TRRS, card detect, and power filtering.
Parts:
- removed J3: Conn_01x03, SparkFun-Connector:1x03
- removed kibuzzard-673EAE78: G***, kibuzzard-673EAE78
- added C4: 10uF, SparkFun-Capacitor:C_0603_1608Metric, F.Cu at (156.2, 96.2)
- added C5: 10uF, SparkFun-Capacitor:C_0603_1608Metric, F.Cu at (153.7, 96.2)
- added J2: Conn_01x04, SparkFun-Connector:1x04, F.Cu at (151.1, 103.5)
- added JP3: CD, SparkFun-Jumper:Jumper_2_PTH_SMD_Combo-NC, F.Cu at (147.3, 75.6)
- added JP4: BUSY, SparkFun-Jumper:Jumper_2_PTH_SMD_Combo-NC, F.Cu at (147.3, 73.0)
- added JP5: RX, SparkFun-Jumper:Jumper_2_PTH_SMD_Combo-NC, F.Cu at (147.3, 70.5)
- added JP6: TX, SparkFun-Jumper:Jumper_2_PTH_SMD_Combo-NC, F.Cu at (147.3, 67.9)
- added JP7: MIC, SparkFun-Jumper:Jumper_2_NC_Trace, B.Cu at (160.0, 111.4)
- added R7: 10k, SparkFun-Resistor:R_0603_1608Metric, F.Cu at (163.8, 100.0)
- added kibuzzard-6792AB76: G***, kibuzzard-6792AB76, F.Cu at (151.1, 100.0)
- added kibuzzard-6792AB99: G***, kibuzzard-6792AB99, B.Cu at (156.8, 111.4)
- added kibuzzard-6792ACE3: G***, kibuzzard-6792ACE3, F.Cu at (140.7, 75.6)
- added kibuzzard-6792ACFA: G***, kibuzzard-6792ACFA, F.Cu at (150.8, 67.9)
- added kibuzzard-6792ACFE: G***, kibuzzard-6792ACFE, F.Cu at (150.8, 70.5)
- added kibuzzard-6792AD08: G***, kibuzzard-6792AD08, F.Cu at (151.8, 73.0)
- added kibuzzard-6792AD10: G***, kibuzzard-6792AD10, F.Cu at (150.8, 75.6)
Connections:
- B1 pad D2: MY_TX -> Net-(JP6-A)
- B1 pad D3: MY_RX -> Net-(B1-*D3)
- B1 pad D4: BUSY -> Net-(JP4-A)
- B1 pad D5: unconnected-(B1-*D5-PadD5) -> Net-(B1-*D5)
- J1 pad R1: DAC_R -> Net-(J2-Pin_3)
- J1 pad S: GND -> Net-(JP7-B)
- J1 pad T: DAC_L -> Net-(J2-Pin_2)
- J6 pad 9: unconnected-(J6-~{DET}-Pad9) -> ~{CARD_DET}
Routing:
- net ~{CARD_DET}: track 0.00 -> 41.1 mm, vias 0 -> 3
- net VCC: track 20.5 -> 42.4 mm, vias 2 -> 3
- net DAC_R: track 20.8 -> 3.62 mm
- net Net-(J2-Pin_3): track 0.00 -> 15.7 mm
- net Net-(J2-Pin_2): track 0.00 -> 10.6 mm
- net DAC_L: track 23.3 -> 13.7 mm, vias 1 -> 2
- net Net-(JP6-A): track 0.00 -> 8.26 mm
- net Net-(JP4-A): track 0.00 -> 8.26 mm
- net Net-(B1-*D3): track 0.00 -> 8.26 mm
- net unconnected-(B1-PadA5/SCL): track 84.4 -> 92.5 mm, vias 1 -> 0
- net MY_RX: track 29.9 -> 21.8 mm
- net Net-(B1-*D5): track 0.00 -> 8.06 mm
- net MY_TX: track 38.8 -> 30.9 mm
- net BUSY: track 44.1 -> 38.1 mm
- net unconnected-(B1-PadA4/SDA): track 80.7 -> 86.1 mm, vias 1 -> 0
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